File: kep-643/kep-643.kicad_sch (KiCad schematic)
At the start: 32 parts, among them J2 CN7, J3 CN8, J4 CN7, J5 CN6, SW1 Function, SW2 Play / Stop, SW3 Rec, SW4 Lesson, SW5 Piano, SW6 E. Piano / Organ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

Commit message: Add the linked connectors. Add the labels.
Parts:
- added J1: CN6, symbol Connector_Generic:Conn_01x13
- added J6: CN11, symbol Connector_Generic:Conn_01x13
Connections:
- new net: J1.1 (Pin_1), J6.1 (Pin_1)
- new net: J1.10 (Pin_10), J6.10 (Pin_10)
- new net: J1.11 (Pin_11), J6.11 (Pin_11)
- new net: J1.12 (Pin_12), J6.12 (Pin_12)
- new net: J1.13 (Pin_13), J6.13 (Pin_13)
- new net: J1.2 (Pin_2), J6.2 (Pin_2)
- new net: J1.3 (Pin_3), J6.3 (Pin_3)
- new net: J1.4 (Pin_4), J6.4 (Pin_4)
- new net: J1.5 (Pin_5), J6.5 (Pin_5)
- new net: J1.6 (Pin_6), J6.6 (Pin_6)
- new net: J1.7 (Pin_7), J6.7 (Pin_7)
- new net: J1.8 (Pin_8), J6.8 (Pin_8)
- new net: J1.9 (Pin_9), J6.9 (Pin_9)
