File: kep-692/kep-692.kicad_sch (KiCad schematic)
At the start: 18 parts, among them CN11 Conn_01x13, CN7 Conn_01x15, U1 HC541, U2 LV541

Commit message: Add the linked connectors. Add the labels.
Parts:
- added J1: CN6, symbol Connector_Generic:Conn_01x13
- added J2: CN11, symbol Connector_Generic:Conn_01x13
Connections:
- new net: J1.1 (Pin_1), J2.1 (Pin_1)
- new net: J1.10 (Pin_10), J2.10 (Pin_10)
- new net: J1.11 (Pin_11), J2.11 (Pin_11)
- new net: J1.12 (Pin_12), J2.12 (Pin_12)
- new net: J1.13 (Pin_13), J2.13 (Pin_13)
- new net: J1.2 (Pin_2), J2.2 (Pin_2)
- new net: J1.3 (Pin_3), J2.3 (Pin_3)
- new net: J1.4 (Pin_4), J2.4 (Pin_4)
- new net: J1.5 (Pin_5), J2.5 (Pin_5)
- new net: J1.6 (Pin_6), J2.6 (Pin_6)
- new net: J1.7 (Pin_7), J2.7 (Pin_7)
- new net: J1.8 (Pin_8), J2.8 (Pin_8)
- new net: J1.9 (Pin_9), J2.9 (Pin_9)
Other:
- note added: "PWR_BTN"
- note added: "VOL_OUT"

Commit message: Add op-amps, missing connectors.
Parts:
- added CN10: Conn_01x07, symbol Connector_Generic:Conn_01x07
- added CN2: Conn_01x04, symbol Connector_Generic:Conn_01x04
- added CN3: Conn_01x06, symbol Connector_Generic:Conn_01x06
- added CN5: Conn_01x10, symbol Connector_Generic:Conn_01x10
- added CN9: Conn_01x05, symbol Connector_Generic:Conn_01x05
- added U3: NJM4580, symbol Amplifier_Operational:NJM4580
Other:
- note added: "3 pedal port"
- note added: "5v"
- note added: "Audio Port"
- note added: "Debug port"
- note added: "MIDI port"
- note added: "Speaker port"
- moved on the sheet: CN11, CN7, J1, J2, R77, R78, R79, R80, R82, R83, R84, R85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

Commit message: Add Labels to CN10.
Other:
- note added: "Damper"
- note added: "This is connected to something."
- note added: "To CN1 (KEP-641) via blue cable"
- note added: "To CN3 (KEP-641) via purple cable"
Changed lines of the file:
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@@
+		)
+	)
+	(text "+5v"
+		(exclude_from_sim no)
+		(at 36.068 113.284 0)
+		(effects
+			(font
+				(size 1.27 1.27)
+			)
 		)
 	)
@@
 		)
 	)
+	(text "This is connected to something."
+		(exclude_from_sim no)
+		(at 799.846 322.834 0)
+		(effects
+			(font
+				(size 1.27 1.27)
+			)
+		)
+	)
 	(text "KD5 (S2)"
 		(exclude_from_sim no)
@@
 		)
 	)
+	(text "Damper"
+		(exclude_from_sim no)
+		(at 787.908 327.914 0)
+		(effects
+			(font
+				(size 1.27 1.27)
+			)
+		)
+	)
 	(text "Debug port"
 		(exclude_from_sim no)
@@
 		)
 	)
+	(text "To CN1 (KEP-641)\nvia blue cable "
+		(exclude_from_sim no)
+		(at 41.148 139.446 0)
+		(effects
+			(font
+				(size 1.27 1.27)
+			)
+		)
+	)
 	(text "SA2"
 		(exclude_from_sim no)
@@
 		)
 	)
+	(text "Damper"
+		(exclude_from_sim no)
+		(at 787.908 325.374 0)
+		(effects
+			(font
+				(size 1.27 1.27)
+			)
+		)
+	)
 	(text "GND"
 		(exclude_from_sim no)
@@
 		(effects
 			(font
+				(size 1.27 1.27)
+			)
+		)
+	)
+	(text "To CN3 (KEP-641)\nvia purple cable"
+		(exclude_from_sim no)
+		(at 784.098 344.17 0)
+		(effects
+			(font
